Commit message: updated stub script, team param, detector

File: ros/meam520_labs/urdf/turntable.xacro (robot description, xacro)
@@ -73,5 +73,10 @@
   </gazebo>
   <gazebo reference="upper_base">
-    <material>Gazebo/LightGrey</material>
+    <material>
+      <ambient>.8 .8 .8 1</ambient>
+      <diffuse>.8 .8 .8 1</diffuse>
+      <specular>.8 .8 .8 1</specular>
+      <emissive>0 0 0 0</emissive>
+    </material>
     <collision>
       <surface>
