Commit message: Added some changes based on kod*lab experience

File: ros/meam520_labs/urdf/cube.xacro (robot description, xacro)
@@ -5,12 +5,12 @@
       <pose>0 0 0 0 0 0</pose>
       <inertial>
-        <mass>0.050</mass>
+        <mass>0.10</mass>
         <inertia>
-          <ixx>0.0002150533</ixx>
+          <ixx>0.002150533</ixx>
           <ixy>0</ixy>
           <ixz>0</ixz>
-          <iyy>0.0002150533</iyy>
+          <iyy>0.002150533</iyy>
           <iyz>0</iyz>
-          <izz>0.0002150533</izz>
+          <izz>0.002150533</izz>
         </inertia>
       </inertial>
@@ -26,11 +26,7 @@
                  according to:
                  http://www.fpl.fs.fed.us/documnts/fplgtr/fplgtr113/ch04.pdf -->
-            <poissons_ratio>0.347</poissons_ratio>
-            <elastic_modulus>8.8e+09</elastic_modulus>
             <ode>
-              <kp>100000</kp>
-              <kd>100</kd>
-              <max_vel>100.0</max_vel>
-              <min_depth>0.001</min_depth>
+              <kp>300000</kp>
+              <kd>1000</kd>
             </ode>
           </contact>
@@ -41,5 +37,13 @@
               <surface_radius>0.0254</surface_radius>
             </torsional>
+            <ode>
+              <mu>2</mu>
+              <mu2>2</mu2>
+            </ode>
           </friction>
+          <bounce>
+            <restitution_coefficient>0</restitution_coefficient>
+             <threshold>1e+06</threshold>
+          </bounce>
         </surface>
       </collision>

File: ros/meam520_labs/urdf/turntable.xacro (robot description, xacro)
@@ -74,4 +74,27 @@
   <gazebo reference="upper_base">
     <material>Gazebo/LightGrey</material>
+    <collision>
+      <surface>
+        <bounce>
+          <restitution_coefficient>0</restitution_coefficient>
+          <threshold>1e+06</threshold>
+        </bounce>
+        <friction>
+          <torsional>
+            <coefficient>100</coefficient>
+          </torsional>
+          <ode>
+            <mu>100</mu>
+            <mu2>100</mu2>
+          </ode>
+        </friction>
+        <contact>
+          <ode>
+            <kp>300000</kp>
+            <kd>1000</kd>
+          </ode>
+        </contact>
+      </surface>
+    </collision>
   </gazebo>
 </robot>

Commit message: tweaking block physics

File: ros/meam520_labs/urdf/cube.xacro (robot description, xacro)
@@ -7,10 +7,10 @@
         <mass>0.10</mass>
         <inertia>
-          <ixx>0.002150533</ixx>
+          <ixx>0.0002150533</ixx>
           <ixy>0</ixy>
           <ixz>0</ixz>
-          <iyy>0.002150533</iyy>
+          <iyy>0.0002150533</iyy>
           <iyz>0</iyz>
-          <izz>0.002150533</izz>
+          <izz>0.0002150533</izz>
         </inertia>
       </inertial>

File: ros/meam520_labs/urdf/turntable.xacro (robot description, xacro)
@@ -12,5 +12,4 @@
     </transmission>
     <xacro:property name="base_radius" value="0.3048" />
-    <!-- <xacro:property name="base_radius" value="0.4572" /> -->
     <xacro:property name="total_height" value="0.02" />
     <link name="world"></link>
@@ -62,5 +61,5 @@
       <child link="upper_base"/>
       <axis xyz="0 0 1"/>
-      <!-- <limit lower="-1.4" upper="1.4" effort="10" velocity="3.67"/> -->
+      <limit lower="-1.4" upper="1.4" effort="10" velocity="3.67"/>
     </joint>
   <gazebo>

Commit message: simulated tag detection and detection visualization

File: ros/meam520_labs/urdf/cube.xacro (robot description, xacro)
@@ -1,6 +1,6 @@
 <?xml version="1.0" ?>
 <sdf version="1.5">
-  <model name="wood_cube_2_5cm">
-    <link name="link">
+  <model name="wood_cube_5cm">
+    <link name="block">
       <pose>0 0 0 0 0 0</pose>
       <inertial>
@@ -55,10 +55,4 @@
           </box>
         </geometry>
-        <!-- <material>
-          <script>
-            <uri>file://media/materials/scripts/gazebo.material</uri>
-            <name>Gazebo/Wood</name>
-          </script>
-        </material> -->
         <material>
           <ambient>$(arg color)</ambient>
@@ -67,7 +61,85 @@
           <emissive>0 0 0 0</emissive>
         </material>
-    </visual>
+      </visual>
+    </link>
+    <link name="tag1">
+      <inertial>
+        <mass>0.001</mass>
+        <inertia>
+          <ixx>0.00000000001</ixx>
+          <ixy>0</ixy>
+          <ixz>0</ixz>
+          <iyy>0.00000000001</iyy>
+          <iyz>0</iyz>
+          <izz>0.00000000001</izz>
+        </inertia>
+      </inertial>
+    </link>
+    <link name="tag2">
+      <inertial>
+        <mass>0.001</mass>
+        <inertia>
+          <ixx>0.00000000001</ixx>
+          <ixy>0</ixy>
+          <ixz>0</ixz>
+          <iyy>0.00000000001</iyy>
+          <iyz>0</iyz>
+          <izz>0.00000000001</izz>
+        </inertia>
+      </inertial>
+    </link>
+    <link name="tag3">
+      <inertial>
+        <mass>0.001</mass>
+        <inertia>
+          <ixx>0.00000000001</ixx>
+          <ixy>0</ixy>
+          <ixz>0</ixz>
+          <iyy>0.00000000001</iyy>
+          <iyz>0</iyz>
+          <izz>0.00000000001</izz>
+        </inertia>
+      </inertial>
+    </link>
+    <link name="tag4">
+      <inertial>
+        <mass>0.001</mass>
+        <inertia>
+          <ixx>0.00000000001</ixx>
+          <ixy>0</ixy>
+          <ixz>0</ixz>
+          <iyy>0.00000000001</iyy>
+          <iyz>0</iyz>
+          <izz>0.00000000001</izz>
+        </inertia>
+      </inertial>
+    </link>
+    <link name="tag5">
+      <inertial>
+        <mass>0.001</mass>
+        <inertia>
+          <ixx>0.00000000001</ixx>
+          <ixy>0</ixy>
+          <ixz>0</ixz>
+          <iyy>0.00000000001</iyy>
+          <iyz>0</iyz>
+          <izz>0.00000000001</izz>
+        </inertia>
+      </inertial>
+    </link>
+    <link name="tag6">
+      <inertial>
+        <mass>0.001</mass>
+        <inertia>
+          <ixx>0.00000000001</ixx>
+          <ixy>0</ixy>
+          <ixz>0</ixz>
+          <iyy>0.00000000001</iyy>
+          <iyz>0</iyz>
+          <izz>0.00000000001</izz>
+        </inertia>
+      </inertial>
       <visual name="marked">
-        <pose>0 0 0.0254 0 0 0</pose>
+        <pose>0 0 0.02542 0 0 0</pose>
         <geometry>
           <box>
@@ -83,4 +155,47 @@
       </visual>
     </link>
+    <joint name="tag1_joint" type="fixed">
+      <parent>block</parent>
+      <child>tag1</child>
+      <pose>.0254 0 0 1.5708 0 1.5708</pose>
+      <preserveFixedJoint>true</preserveFixedJoint>
+    </joint>
+    <joint name="tag2_joint" type="fixed">
+      <parent>block</parent>
+      <child>tag2</child>
+      <pose>0 .0254 0 1.5708 0 3.14159</pose>
+      <preserveFixedJoint>true</preserveFixedJoint>
+    </joint>
+    <joint name="tag3_joint" type="fixed">
+      <parent>block</parent>
+      <child>tag3</child>
+      <pose>-.0254 0 0 1.5708 0 -1.5708</pose>
+      <preserveFixedJoint>true</preserveFixedJoint>
+    </joint>
+    <joint name="tag4_joint" type="fixed">
+      <parent>block</parent>
+      <child>tag4</child>
+      <pose>0 -.0254 0 1.5708 0 0</pose>
+      <preserveFixedJoint>true</preserveFixedJoint>
+    </joint>
+    <joint name="tag5_joint" type="fixed">
+      <parent>block</parent>
+      <child>tag5</child>
+      <pose>0 0 -.0254 0 3.14159 -1.5708</pose>
+      <preserveFixedJoint>true</preserveFixedJoint>
+    </joint>
+    <joint name="tag6_joint" type="fixed">
+      <!-- <axis>
+        <xyz>0 0 1</xyz>
+      </axis>
+      <limit>
+        <upper>0</upper>
+        <lower>0</lower>
+      </limit> -->
+      <parent>block</parent>
+      <child>tag6</child>
+      <pose>0 0 .0254 0 0 -1.5708</pose>
+      <preserveFixedJoint>true</preserveFixedJoint>
+    </joint>
   </model>
 </sdf>
