Commit message: fixes due to collision geometry change and detection visualizer

File: ros/meam520_labs/urdf/nogravity.urdf (robot description, URDF)
Before this commit: robot panda, 13 links, 12 joints
Links:
- link panda_link5: geometry collision mesh filename=package://franka_panda_description/meshes/collision/link5.s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; visual mesh filename=package://franka_panda_description/meshes/visual/link5.dae
